Commit message: Add mars urdf to sim
Findings:

High: repeated simulations in the same browser session will start with stale arm/gripper state instead of a clean pose. The frontend intentionally reuses session_id across runs in lib/robot/simulation-client.ts (line 16) and lib/robot/simulation-client.ts (line 46), and the API reuses the existing MarsSimulator in simulation/api/main.py (line 123). But reset_state() only resets base position/trail in simulation/core/mars_sim.py (line 127); it never restores current_joints from simulation/core/mars_sim.py (line 53). After a wave, gripper close, etc., the next simulation will interpolate from the old pose, so the preview no longer matches a fresh run.

High: the new “Simulate 3D” path can silently produce the wrong behavior for many valid Blockly programs. The UI serializes the full workspace in components/exercise/blockly-workspace.tsx (line 205), but process_block_chain() in simulation/api/main.py (line 40) handles only a small subset of statement blocks and completely ignores inputs. By contrast, real execution supports conditionals, loops, value expressions, sensors, and more in lib/robot/executor.ts (line 226), and those blocks are exposed in the toolbox in lib/blockly-config/toolbox.ts (line 58). A program using controls_if, controls_repeat_ext, controls_whileUntil, or mars_wait_until will “simulate” as if those blocks were no-ops, with no warning to the user.

Medium: simulation sessions are never retired, and each new session starts its own gRPC server on a new port. The global sessions map in simulation/api/main.py (line 21) only grows, and creating a MarsSimulator immediately calls serve_grpc() in simulation/core/mars_sim.py (line 27). A reload, a second tab, or multiple users will leave old recording streams and ports alive indefinitely. That looks like a resource leak for any long-running dev server or deployed service.

Open questions / assumptions:

I assumed the simulator is meant to preview the same semantics as “Run on MARS,” because both paths consume BlockExecutor.serializeWorkspace(...).
I did not verify the Python service end-to-end because pytest is not installed in the current shell.
Checks:

npm run typecheck passed.
pytest simulation/tests/test_api.py could not run: pytest: command not found

Signed-off-by: Maxwell Henderson <mxwhenderson@gmail.com>

File: simulation/models/mars_robot.urdf (robot description, URDF)
Before this commit: robot mars_robot, 4 links, 3 joints
Links:
- removed link arm_base
- removed link left_wheel
- removed link right_wheel
- added link arm_camera_link, mass 0.01
- added link camera_optical_frame
- added link ee_link, mass 0.001; visual sphere radius=0.005
- added link head, mass 0.148; visual mesh filename=meshes/head.STL scale=1 1 1
- added link head_camera_left, mass 0.01; visual sphere radius=0.005
- added link head_camera_right, mass 0.01; visual sphere radius=0.005
- added link link1, mass 0.065; visual mesh filename=meshes/link1.STL scale=1 1 1
- added link link2, mass 0.080; visual mesh filename=meshes/link2.STL scale=1 1 1
- added link link3, mass 0.055; visual mesh filename=meshes/link3.STL scale=1 1 1
- added link link4, mass 0.022; visual mesh filename=meshes/link4.STL scale=1 1 1
- added link link5, mass 0.050; visual mesh filename=meshes/link5.STL scale=1 1 1
- added link link61, mass 0.012; visual mesh filename=meshes/link61.STL scale=1 1 1
- added link link62, mass 0.012; visual mesh filename=meshes/link62.STL scale=1 1 1
- added link right_camera_optical_frame
- link base_link: mass None -> 0.89; geometry visual mesh filename=meshes/base.STL scale=1 1 1
Joints:
- removed joint base_to_arm_base
- removed joint base_to_left_wheel
- removed joint base_to_right_wheel
- added joint ee_joint: type fixed, parent link5, child ee_link, origin xyz=0.091838 0 0 rpy=0 0 0
- added joint fixed_arm_camera_link: type fixed, parent link5, child arm_camera_link, origin xyz=0.03378 0 0.05052 rpy=0 0.43633 0
- added joint fixed_camera_optical_frame: type fixed, parent head_camera_left, child camera_optical_frame, origin xyz=0 0 0 rpy=-1.5708 0 -1.5708
- added joint fixed_head_camera_left: type fixed, parent head, child head_camera_left, origin xyz=0.04327 0.0297 -0.000275 rpy=0 0 0
- added joint fixed_head_camera_right: type fixed, parent head, child head_camera_right, origin xyz=0.04327 -0.0303 -0.000275 rpy=0 0 0
- added joint fixed_right_camera_optical_frame: type fixed, parent head_camera_right, child right_camera_optical_frame, origin xyz=0 0 0 rpy=-1.5708 0 -1.5708
- added joint joint1: type revolute, parent base_link, child link1, origin xyz=0.086 -0.05285 0.04025 rpy=0 0 0, axis 0 0 1, limit lower=-1.5708 upper=1.5708 effort=2.0 velocity=2.0
- added joint joint2: type revolute, parent link1, child link2, origin xyz=0 0 0.04425 rpy=0 0 0, axis 0 1 0, limit lower=-1.5708 upper=1.22 effort=2.0 velocity=2.0
- added joint joint3: type revolute, parent link2, child link3, origin xyz=0.02825 0 0.12125 rpy=0 0 0, axis 0 1 0, limit lower=-1.5708 upper=1.7453 effort=2.0 velocity=2.0
- added joint joint4: type revolute, parent link3, child link4, origin xyz=0.1375 0 0.0045 rpy=0 0 0, axis 0 1 0, limit lower=-1.9199 upper=1.7453 effort=2.0 velocity=2.0
- added joint joint5: type revolute, parent link4, child link5, origin xyz=0.019 0 0 rpy=0 0 0, axis 1 0 0, limit lower=-1.5708 upper=1.5708 effort=2.0 velocity=2.0
- added joint joint6: type revolute, parent link5, child link61, origin xyz=0.044 -0.0092 0 rpy=0 0 0, axis 0 0 -1, limit lower=-0.8727 upper=0.3491 effort=2.0 velocity=2.0
- added joint joint6M: type revolute, parent link5, child link62, origin xyz=0.044 0.0091 0 rpy=0 0 0, axis 0 0 -1, limit lower=-0.8727 upper=0.3491 effort=2.0 velocity=2.0, mimic joint=joint6 multiplier=-1 offset=0
- added joint joint_head: type revolute, parent base_link, child head, origin xyz=-0.040751 -0.0002 0.25882 rpy=0 0 0, axis 0 -1 0, limit lower=-0.1745 upper=0.5236 effort=2.0 velocity=2.0
